Commit message: final

File: dobbie_ws/src/descy/urdf/dobbie.urdf.xacro (robot description, xacro)
@@ -25,5 +25,5 @@
               rpy="-2.962441408225233 -1.5680409623316962 -1.7467263101041604"/>
       <geometry>
-        <mesh filename="${mesh_path}/converted_base_mesh.stl"/>
+        <mesh filename="${mesh_path}/base_mesh.stl"/>
       </geometry>
       <material name="white"/>
@@ -33,5 +33,5 @@
               rpy="-2.962441408225233 -1.5680409623316962 -1.7467263101041604"/>
       <geometry>
-        <mesh filename="${mesh_path}/converted_base_mesh.stl"/>
+        <mesh filename="${mesh_path}/base_mesh.stl"/>
       </geometry>
     </collision>
@@ -56,5 +56,5 @@
               rpy="-1.5652545899663657 -1.518025120993771 -1.5759784889015487"/>
       <geometry>
-        <mesh filename="${mesh_path}/converted_link1_mesh.stl"/>
+        <mesh filename="${mesh_path}/link1_mesh.stl"/>
       </geometry>
       <material name="white"/>
@@ -64,5 +64,5 @@
               rpy="-1.5652545899663657 -1.518025120993771 -1.5759784889015487"/>
       <geometry>
-        <mesh filename="${mesh_path}/converted_link1_mesh.stl"/>
+        <mesh filename="${mesh_path}/link1_mesh.stl"/>
       </geometry>
     </collision>
@@ -90,5 +90,5 @@
               rpy="0.05365179981860118 -0.008747444451175479 0.06403379882506219"/>
       <geometry>
-        <mesh filename="${mesh_path}/converted_link2_mesh.stl"/>
+        <mesh filename="${mesh_path}/link2_mesh.stl"/>
       </geometry>
       <material name="white"/>
@@ -98,5 +98,5 @@
               rpy="0.05365179981860118 -0.008747444451175479 0.06403379882506219"/>
       <geometry>
-        <mesh filename="${mesh_path}/converted_link2_mesh.stl"/>
+        <mesh filename="${mesh_path}/link2_mesh.stl"/>
       </geometry>
     </collision>
@@ -124,5 +124,5 @@
               rpy="1.6580773132277526 0.00011419959347480635 0.00016929457412240279"/>
       <geometry>
-        <mesh filename="${mesh_path}/converted_link3_mesh.stl"/>
+        <mesh filename="${mesh_path}/link3_mesh.stl"/>
       </geometry>
       <material name="white"/>
@@ -132,5 +132,5 @@
               rpy="1.6580773132277526 0.00011419959347480635 0.00016929457412240279"/>
       <geometry>
-        <mesh filename="${mesh_path}/converted_link3_mesh.stl"/>
+        <mesh filename="${mesh_path}/link3_mesh.stl"/>
       </geometry>
     </collision>
@@ -158,5 +158,5 @@
               rpy="1.3881086882909015 0.003921029036773049 0.0007426984677866288"/>
       <geometry>
-        <mesh filename="${mesh_path}/converted_link4_mesh.stl"/>
+        <mesh filename="${mesh_path}/link4_mesh.stl"/>
       </geometry>
       <material name="white"/>
@@ -166,5 +166,5 @@
               rpy="1.3881086882909015 0.003921029036773049 0.0007426984677866288"/>
       <geometry>
-        <mesh filename="${mesh_path}/converted_link4_mesh.stl"/>
+        <mesh filename="${mesh_path}/link4_mesh.stl"/>
       </geometry>
     </collision>
@@ -192,5 +192,5 @@
               rpy="-0.03931949901759166 5.812106912839177e-05 0.011601086068503979"/>
       <geometry>
-        <mesh filename="${mesh_path}/converted_link5_mesh.stl"/>
+        <mesh filename="${mesh_path}/link5_mesh.stl"/>
       </geometry>
       <material name="white"/>
@@ -200,5 +200,5 @@
               rpy="-0.03931949901759166 5.812106912839177e-05 0.011601086068503979"/>
       <geometry>
-        <mesh filename="${mesh_path}/converted_link5_mesh.stl"/>
+        <mesh filename="${mesh_path}/link5_mesh.stl"/>
       </geometry>
     </collision>
